File: board/board.kicad_pcb (KiCad board)
At the start: 2 copper layers, 21 x 13 mm, 1 part

Commit message: initial
Parts:
- removed LOGO1: Logo_Open_Hardware_Small, Symbol:OSHW-Symbol_6.7x6mm_SilkScreen
- added C1: 22nF, Capacitor_SMD:C_0603_1608Metric, F.Cu at (115.4, 76.1)
- added C10: 10nF, Capacitor_SMD:C_0603_1608Metric, B.Cu at (86.2, 100.8)
- added C11: 4.7u, Capacitor_SMD:C_0603_1608Metric, B.Cu at (89.2, 100.8)
- added C12: 18pF, Capacitor_SMD:C_0603_1608Metric, B.Cu at (79.2, 90.0)
- added C13: 18pF, Capacitor_SMD:C_0603_1608Metric, B.Cu at (79.2, 96.2)
- added C14: 6.8nF, Capacitor_SMD:C_0603_1608Metric, F.Cu at (111.9, 86.5)
- added C15: 10nF, Capacitor_SMD:C_0603_1608Metric, F.Cu at (114.8, 82.4)
- added C2: 6.8nF, Capacitor_SMD:C_0603_1608Metric, F.Cu at (111.9, 85.0)
- added C3: 1uF, Capacitor_SMD:C_0603_1608Metric, B.Cu at (90.8, 85.7)
- added C4: 100nF, Capacitor_SMD:C_0603_1608Metric, B.Cu at (97.0, 92.0)
- added C5: 100nF, Capacitor_SMD:C_0603_1608Metric, B.Cu at (81.7, 97.0)
- added C6: 100nF, Capacitor_SMD:C_0603_1608Metric, B.Cu at (87.8, 100.8)
- added C7: 100nF, Capacitor_SMD:C_0603_1608Metric, B.Cu at (97.0, 95.2)
- added C8: 100nF, Capacitor_SMD:C_0603_1608Metric, B.Cu at (90.8, 100.8)
- added C9: 100nF, Capacitor_SMD:C_0603_1608Metric, B.Cu at (96.0, 98.7)
- added J1: 002_SPI, on_edge:on_edge_2x05_device, F.Cu at (77.0, 80.5)
- added J2: Conn_01x02_Male, Connector_PinHeader_2.54mm:PinHeader_1x02_P2.54mm_Vertical, B.Cu at (79.7, 100.8)
- added J3: 019_100BASE-T_with_CT, on_edge:on_edge_2x05_host, F.Cu at (122.0, 80.5)
- added R1: 12.4k, Resistor_SMD:R_0603_1608Metric, B.Cu at (100.7, 98.5)
- added R10: 3.3R, Resistor_SMD:R_0603_1608Metric, F.Cu at (108.7, 80.0)
- added R11: 3.3R, Resistor_SMD:R_0603_1608Metric, F.Cu at (108.7, 78.5)
- added R2: 1M, Resistor_SMD:R_0603_1608Metric, B.Cu at (79.2, 93.1)
- added R3: 10R, Resistor_SMD:R_0805_2012Metric, F.Cu at (113.6, 75.9)
- added R4: 49.9R, Resistor_SMD:R_0805_2012Metric, F.Cu at (109.9, 76.0)
- added R5: 49.9R, Resistor_SMD:R_0805_2012Metric, F.Cu at (107.9, 76.0)
- added R6: 49.9R, Resistor_SMD:R_0805_2012Metric, F.Cu at (113.1, 82.5)
- added R7: 49.9R, Resistor_SMD:R_0805_2012Metric, F.Cu at (111.1, 82.5)
- added R8: 3.3R, Resistor_SMD:R_0603_1608Metric, F.Cu at (109.0, 86.5)
- added R9: 3.3R, Resistor_SMD:R_0603_1608Metric, F.Cu at (108.9, 85.0)
- added U1: W5500, Package_QFP:LQFP-48_7x7mm_P0.5mm, B.Cu at (90.0, 93.7)
- added Y1: 25MHz, Crystal:Crystal_SMD_5032-2Pin_5.0x3.2mm, B.Cu at (82.0, 93.0)
Routing:
- net GND: track 0.00 -> 182.8 mm, vias 0 -> 22
- net +3V3: track 0.00 -> 94.0 mm, vias 0 -> 5
- net /controller/SS: track 0.00 -> 21.3 mm
- net Net-(U1-Pad2): track 0.00 -> 19.6 mm, vias 0 -> 1
- net /controller/MOSI: track 0.00 -> 18.6 mm, vias 0 -> 1
- net Net-(U1-Pad1): track 0.00 -> 18.3 mm, vias 0 -> 1
- net Net-(U1-Pad6): track 0.00 -> 18.0 mm, vias 0 -> 1
- net Net-(U1-Pad5): track 0.00 -> 16.7 mm, vias 0 -> 1
- net /controller/MISO: track 0.00 -> 16.7 mm, vias 0 -> 1
- net /controller/SCLK: track 0.00 -> 16.5 mm, vias 0 -> 1
- net /controller/~reset: track 0.00 -> 16.2 mm, vias 0 -> 2
- net /controller/TXN: track 0.00 -> 14.4 mm
- net /controller/TXP: track 0.00 -> 12.4 mm
- net /controller/INT: track 0.00 -> 12.4 mm, vias 0 -> 1
- net /controller/CT2: track 0.00 -> 9.74 mm, vias 0 -> 1
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- added copper zone on B.Cu, net +3V3
- added copper zone on F.Cu, net GND
Other:
- board size 21 x 13 mm -> 45 x 29 mm
- rule pad_to_mask_clearance: 0 -> 0.04
- board text added: "osf.002.v0.1"
- board text added: "osf.b078.v1.0"
