File: board/board.kicad_sch (KiCad schematic)
At the start: 1 part

Commit message: initial
Parts:
- removed LOGO1: Logo_Open_Hardware_Small, Symbol:OSHW-Symbol_6.7x6mm_SilkScreen, symbol Graphic:Logo_Open_Hardware_Small
- added C3: 1uF, Capacitor_SMD:C_0603_1608Metric, symbol Device:C_Small
- added C4: 100nF, Capacitor_SMD:C_0603_1608Metric, symbol Device:C_Small
- added J1: 002_SPI, on_edge:on_edge_2x05_device, symbol put_on_edge:002_SPI
- added J2: Conn_01x02_Male, Connector_PinHeader_2.54mm:PinHeader_1x02_P2.54mm_Vertical, symbol Connector:Conn_01x02_Male
- added J3: 019_100BASE-T_with_CT, on_edge:on_edge_2x05_host, symbol put_on_edge:019_100BASE-T_with_CT
Connections:
- new net +3V3: C3.1, C4.1, J1.9 (3.3V)
- new net GND: C3.2, C4.2, J1.1 (GND), J3.1 (GND), J3.6 (GND)
- new net controller/CT1: J3.7 (CT1)
- new net controller/CT2: J3.8 (CT2)
- new net controller/DUPLED: J2.1 (Pin_1)
- new net controller/INT: J1.5 (INT)
- new net controller/MISO: J1.3 (MISO)
- new net controller/MOSI: J1.2 (MOSI)
- new net controller/RXN: J3.5 (TD2-)
- new net controller/RXP: J3.4 (TD2+)
- new net controller/SCLK: J1.4 (SCLK)
- new net controller/SPDLED: J2.2 (Pin_2)
- new net controller/SS: J1.6 (CS)
- new net controller/TXN: J3.3 (TD1-)
- new net controller/TXP: J3.2 (TD1+)
- new net controller/~reset: J1.8 (~{RESET})
- no-connect marks 0 -> 2
Other:
- removed sheet implementation
- added sheet controller (controller.kicad_sch)
- note removed: "Input connectors go here"
- note removed: "Output connectors go here"
